Commit message: Add SLSQP-based motion retargeting

File: examples_pybullet/assets/shadow_hand/model.urdf (robot description, URDF)
Before this commit: robot shadow_hand, 25 links, 24 joints
Links:
- link index_finger_distal: mass None -> 0.5
- link index_finger_knuckle: mass None -> 0.5
- link index_finger_middle: mass None -> 0.5
- link index_finger_proximal: mass None -> 0.5
- link little_finger_distal: mass None -> 0.5
- link little_finger_knuckle: mass None -> 0.5
- link little_finger_metacarpal: mass None -> 0.5
- link little_finger_middle: mass None -> 0.5
- link little_finger_proximal: mass None -> 0.5
- link middle_finger_distal: mass None -> 0.5
- link middle_finger_knuckle: mass None -> 0.5
- link middle_finger_middle: mass None -> 0.5
- link middle_finger_proximal: mass None -> 0.5
- link palm: mass None -> 0.5
- link ring_finger_distal: mass None -> 0.5
- link ring_finger_knuckle: mass None -> 0.5
- link ring_finger_middle: mass None -> 0.5
- link ring_finger_proximal: mass None -> 0.5
- link thumb_distal: mass None -> 0.5
- link thumb_middle: mass None -> 0.5
- link thumb_proximal: mass None -> 0.5
- link wrist: mass None -> 0.5
